File: stusb.kicad_sch (KiCad schematic)
At the start: 25 parts, among them J1 USB_C_Receptacle_USB2.0, Q1 DTC143E, Q2 DTC143E, Q3 DTC143E, Q4 IRF8736, U2 FUSB307B, U3 FT230XQ

Commit message: transistor oops
Connections:
- net GND: now also Q3.2 (E); no longer Q3.3 (C)
- net at R6.2: now also Q3.3 (C); no longer Q3.2 (E)
Changed lines of the file:
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@@
     (pin "3")
   )
-  (symbol (lib_id "-Discrete:DTC143E") (at 194.31 55.88 0) (mirror x) (unit 1)
+  (symbol (lib_id "-Discrete:DTC143E") (at 194.31 55.88 0) (unit 1)
     (in_bom yes) (on_board yes)
-    (property "Reference" "Q3" (id 0) (at 199.0852 57.0484 0)
+    (property "Reference" "Q3" (id 0) (at 199.0852 54.7116 0)
       (effects (font (size 1.27 1.27)) (justify left))
     )
-    (property "Value" "DTC143E" (id 1) (at 199.0852 54.737 0)
+    (property "Value" "DTC143E" (id 1) (at 199.0852 57.023 0)
       (effects (font (size 1.27 1.27)) (justify left))
     )

Commit message: drc fixes
Parts:
- removed Q3: DTC143E, Package_TO_SOT_SMD:SOT-323_SC-70, symbol -Discrete:DTC143E
- added Q3: BC858W, Package_TO_SOT_SMD:SOT-323_SC-70, symbol Transistor_BJT:BC858W
Connections:
- net GND: now also Q3.3 (C)
- net SNK: now also Q3.1 (B)
- net at R6.2: now also Q3.2 (E)
Changed lines of the file:
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@@
+    (stroke (width 0) (type default) (color 0 0 0 0))
+  )
+  (wire (pts (xy 161.29 55.88) (xy 189.23 55.88))
     (stroke (width 0) (type default) (color 0 0 0 0))
   )
@@
   (wire (pts (xy 186.69 151.13) (xy 195.58 151.13))
     (stroke (width 0) (type solid) (color 0 0 0 0))
-  )
-  (wire (pts (xy 187.96 55.88) (xy 161.29 55.88))
-    (stroke (width 0) (type default) (color 0 0 0 0))
   )
   (wire (pts (xy 189.5334 76.8262) (xy 191.77 76.8262))
@@
     (pin "1")
     (pin "2")
+  )
+  (symbol (lib_id "Transistor_BJT:BC858W") (at 194.31 55.88 0) (mirror x) (unit 1)
+    (in_bom yes) (on_board yes) (fields_autoplaced)
+    (property "Reference" "Q3" (id 0) (at 199.1615 54.9715 0)
+      (effects (font (size 1.27 1.27)) (justify left))
+    )
+    (property "Value" "BC858W" (id 1) (at 199.1615 57.7466 0)
+      (effects (font (size 1.27 1.27)) (justify left))
+    )
+    (property "Footprint" "Package_TO_SOT_SMD:SOT-323_SC-70" (id 2) (at 199.39 53.975 0)
+      (effects (font (size 1.27 1.27) italic) (justify left) hide)
+    )
+    (property "Datasheet" "http://www.infineon.com/dgdl/Infineon-BC857SERIES_BC858SERIES_BC859SERIES_BC860SERIES-DS-v01_01-en.pdf?fileId=db3a304314dca389011541da0e3a1661" (id 3) (at 194.31 55.88 0)
+      (effects (font (size 1.27 1.27)) (justify left) hide)
+    )
+    (pin "1")
+    (pin "2")
+    (pin "3")
   )
   (symbol (lib_id "Transistor_FET:FDS9435A") (at 181.61 27.94 270) (mirror x) (unit 1)
@@
       (effects (font (size 1.27 1.27)) (justify left) hide)
     )
-    (pin "1")
-    (pin "2")
-    (pin "3")
-  )
-  (symbol (lib_id "-Discrete:DTC143E") (at 194.31 55.88 0) (unit 1)
-    (in_bom yes) (on_board yes)
-    (property "Reference" "Q3" (id 0) (at 199.0852 54.7116 0)
-      (effects (font (size 1.27 1.27)) (justify left))
-    )
-    (property "Value" "DTC143E" (id 1) (at 199.0852 57.023 0)
-      (effects (font (size 1.27 1.27)) (justify left))
-    )
-    (property "Footprint" "Package_TO_SOT_SMD:SOT-323_SC-70" (id 2) (at 194.31 55.88 0)
-      (effects (font (size 1.27 1.27)) (justify left) hide)
-    )
-    (property "Datasheet" "" (id 3) (at 194.31 55.88 0)
-      (effects (font (size 1.27 1.27)) (justify left) hide)
-    )
