File: ws28xx-FUSB307B.kicad_pcb (KiCad board)
At the start: 4 copper layers, 63.5 x 23.3 mm, 77 parts, among them J1 USB_C_Receptacle_USB2.0, Q1 DTC143E, Q2 DTC143E, Q3 DTC143E, Q4 IRF8736, SW1 en, SW2 io0, U1 TXB0102, U2 FUSB307B, U3 FT230XQ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

Commit message: transistor oops
Parts:
- moved R6 0.24 mm to (119.3, 98.3)
Connections:
- Q3 pad 2: Net-(Q3-Pad2) -> GND
- Q3 pad 3: GND -> Net-(R6-Pad2)
- R6 pad 2: Net-(Q3-Pad2) -> Net-(R6-Pad2)
Routing:
- net Net-(R6-Pad2): track 0.00 -> 3.44 mm
- net Net-(Q3-Pad2): track 1.03 -> 0.00 mm
- net GND: vias 89 -> 90
Changed lines of the file:
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@@
   (net 62 "unconnected-(U6-Pad6)")
   (net 63 "unconnected-(U6-Pad21)")
-  (net 64 "Net-(Q3-Pad2)")
+  (net 64 "Net-(R6-Pad2)")
   (footprint "Diode_SMD:D_SMA" (layer "F.Cu")
     (at 143.075 101.4 90)
@@
       (net 57 "SNK") (pinfunction "B") (pintype "input"))
     (pad "2" smd rect locked (at -1 0.65 90) (size 0.45 0.7) (layers "F.Cu" "F.Paste" "F.Mask")
-      (net 64 "Net-(Q3-Pad2)") (pinfunction "E") (pintype "passive"))
+      (net 26 "GND") (pinfunction "E") (pintype "passive"))
     (pad "3" smd rect locked (at 1 0 90) (size 0.45 0.7) (layers "F.Cu" "F.Paste" "F.Mask")
-      (net 26 "GND") (pinfunction "C") (pintype "passive"))
+      (net 64 "Net-(R6-Pad2)") (pinfunction "C") (pintype "passive"))
     (model "${KICAD6_3DMODEL_DIR}/Package_TO_SOT_SMD.3dshapes/SOT-323_SC-70.wrl"
       (offset (xyz 0 0 0))
@@
   )
   (footprint "Resistor_SMD:R_0603_1608Metric" (layer "F.Cu")
-    (at 119.320976 98.542476 -90)
+    (at 119.320976 98.298 -90)
     (descr "Resistor SMD 0603 (1608 Metric), square (rectangular) end terminal, IPC_7351 nominal, (Body size source: IPC-SM-782 page 72, https://www.pcb-3d.com/wordpress/wp-content/uploads/ipc-sm-782a_amendment_1_and_2.pdf), generated with kicad-footprint-generator")
     (tags "resistor")
@@
       (net 32 "Net-(C8-Pad2)") (pintype "passive"))
     (pad "2" smd roundrect locked (at 0.825 0 270) (size 0.8 0.95) (layers "F.Cu" "F.Paste" "F.Mask") (roundrect_rratio 0.25)
-      (net 64 "Net-(Q3-Pad2)") (pintype "passive"))
+      (net 64 "Net-(R6-Pad2)") (pintype "passive"))
     (model "${KICAD6_3DMODEL_DIR}/Resistor_SMD.3dshapes/R_0603_1608Metric.wrl"
       (offset (xyz 0 0 0))
@@
   (via (at 140.716 89.916) (size 0.6858) (drill 0.3302) (layers "F.Cu" "B.Cu") (net 26))
   (via (at 159.512 92.456) (size 0.6858) (drill 0.3302) (layers "F.Cu" "B.Cu") (net 26))
+  (via (at 119.242719 100.979634) (size 0.6858) (drill 0.3302) (layers "F.Cu" "B.Cu") (net 26))
   (via (at 132.275 93.45) (size 0.6858) (drill 0.3302) (layers "F.Cu" "B.Cu") (net 26))
   (via (at 141.484997 101.388) (size 0.6858) (drill 0.3302) (layers "F.Cu" "B.Cu") (net 26))
@@
   (segment (start 126.941807 83.818201) (end 126.357706 83.2341) (width 0.1778) (layer "B.Cu") (net 31))
   (segment (start 154.178 86.868) (end 153.852797 87.304797) (width 0.1778) (layer "B.Cu") (net 31))
-  (segment (start 118.618 102.87) (end 118.579756 102.831756) (width 0.1778) (layer "F.Cu") (net 32))
-  (segment (start 119.320976 97.717476) (end 119.78686 97.717476) (width 0.1778) (layer "F.Cu") (net 32))
+  (segment (start 120.031336 97.473) (end 120.540699 96.963637) (width 0.1778) (layer "F.Cu") (net 32))
+  (segment (start 119.320976 97.473) (end 120.031336 97.473) (width 0.1778) (layer "F.Cu") (net 32))
   (segment (start 118.364 103.124) (end 118.618 102.87) (width 0.1778) (layer "F.Cu") (net 32))
-  (segment (start 119.78686 97.717476) (end 120.540699 96.963637) (width 0.1778) (layer "F.Cu") (net 32))
+  (segment (start 118.618 100.076) (end 118.753812 99.940188) (width 0.1778) (layer "F.Cu") (net 32))
+  (segment (start 118.753812 99.940188) (end 120.052799 99.940188) (width 0.1778) (layer "F.Cu") (net 32))
   (segment (start 120.841 96.774) (end 120.841 98.724003) (width 0.1778) (layer "F.Cu") (net 32))
-  (segment (start 118.579756 102.831756) (end 118.579756 98.458696) (width 0.1778) (layer "F.Cu") (net 32))
+  (segment (start 120.052799 99.940188) (end 121.054992 98.937995) (width 0.1778) (layer "F.Cu") (net 32))
+  (segment (start 118.618 102.87) (end 118.618 100.076) (width 0.1778) (layer "F.Cu") (net 32))
   (segment (start 117.843 103.124) (end 118.364 103.124) (width 0.1778) (layer "F.Cu") (net 32))
-  (segment (start 118.579756 98.458696) (end 119.320976 97.717476) (width 0.1778) (layer "F.Cu") (net 32))
   (segment (start 134.634997 94.288) (end 133.834997 94.288) (width 0.6096) (layer "F.Cu") (net 36))
   (segment (start 117.205976 91.057021) (end 116.075979 91.057021) (width 0.508) (layer "F.Cu") (net 36))
@@
   (segment (start 131.837925 100.838) (end 133.096 100.838) (width 0.1778) (layer "B.Cu") (net 57))
   (segment (start 131.605885 101.092) (end 131.837925 100.838) (width 0.1778) (layer "B.Cu") (net 57))
-  (segment (start 119.320976 99.367476) (end 119.320976 100.398976) (width 0.1778) (layer "F.Cu") (net 64))
+  (segment (start 118.26288 100.838) (end 118.00888 101.092) (width 0.1778) (layer "F.Cu") (net 64))
+  (segment (start 118.26288 99.706096) (end 118.26288 100.838) (width 0.1778) (layer "F.Cu") (net 64))
+  (segment (start 119.320976 99.123) (end 118.845976 99.123) (width 0.1778) (layer "F.Cu") (net 64))
+  (segment (start 118.00888 101.092) (end 117.364 101.092) (width 0.1778) (layer "F.Cu") (net 64))
+  (segment (start 118.845976 99.123) (end 118.26288 99.706096) (width 0.1778) (layer "F.Cu") (net 64))
   (zone locked (net 1) (net_name "VBUS") (layer "F.Cu") (hatch edge 0.508)
     (connect_pads (clearance 0.2794))

Commit message: drc fixes
Parts:
- Q3: value DTC143E -> BC858W
- moved svg2mod 3.64 mm to (159.0, 86.9), turned to 135 degrees
- moved TP15 0.57 mm to (163.3, 84.6)
- moved svg2mod 0.56 mm to (155.2, 87.1), turned to 135 degrees
- moved svg2mod 0.47 mm to (163.3, 89.4)
- renumbered LEDS2 to IO18, LEDS1 to IO19
Connections:
- Q3 pad 2: GND -> Net-(Q3-Pad2)
- Q3 pad 3: Net-(R6-Pad2) -> GND
- R6 pad 2: Net-(R6-Pad2) -> Net-(Q3-Pad2)
Routing:
- net Net-(R6-Pad2): track 3.44 -> 0.00 mm
- net Net-(JP1-Pad1): track 9.16 -> 10.6 mm
- net Net-(Q3-Pad2): track 0.00 -> 1.34 mm
- net Net-(C11-Pad1): track 13.1 -> 14.2 mm
- net GND: vias 90 -> 89
Other:
- board text added: "IO18"
- board text added: "IO19"
- board text removed: "IO"
